File: Main.sch (EAGLE design)
At the start: 24 parts, among them IC1 PIC16F1939P, J1 EM-506-VERTICAL, Q6 IRFD9210

Commit message: Encrypter work
Parts:
- removed PROG: 22-27-2061-06, con-molex:22-27-2061-06
- removed Q1, Q2, Q3, Q4, Q5, Q7: (no value), SparkFun-DiscreteSemi:TRANSISTOR_NPN2N3904
- removed Q6: IRFD9210, transistor-fet:IRFD9210
- removed U1: (no value), SparkFun-DigitalIC:TXB0104PWRSOIC14
- added IC2: 4052N, 40xx:4052N
- added IC3: 24AA01P, microchip:24AA01P
- added J2: PIC_ICSP_6_PINPOLAR_LOCK, SparkFun-Connectors:PIC_ICSP_6_PINPOLAR_LOCK
- added OTPPGM: (no value), jumper:JP1Q
- added R1: (no value), resistor:R-US_0204/2V
- added U$2: CPC1008N, JSB2:CPC1008N
- DM-EN, DM-RST, LOC-SQ, SOS: value 22-27-2021-02 -> TSW-102-02-S-S; device con-molex:22-27-2021-02 -> con-samtec:TSW-102-02-S-S
- I2C: value 22-27-2021-02 -> 22-27-2031-03; device con-molex:22-27-2021-02 -> con-molex:22-27-2031-03
- RTC1: I2CADDR (none) -> 0xD0
Connections:
- removed net N$25: IC1.RC5/SDO/SEG10, Q5.B
- new net N$27: IC3.WP, OTPPGM.2, R2.1
- new net N$28: IC1.VPP/!MCLR!/RE3, J2.VPP
- net +5V: now also IC2P.VCC, IC3.A0, IC3.A1, IC3.A2, IC3.VCC, J2.VCC, U$2.DC@1; no longer PROG-2.S, Q6.S, U1.VCCB
- net GND: now also DM-EN-2.1, DM-RST-2.1, I2C-3.S, IC2A.INH, IC2P.GND, IC2P.VEE, IC3.GND, J2.GND, LOC-SQ-2.1, OTPPGM.1, RB-INT-1.1, SOS-2.1, U$1.3, U$2.IN-; no longer DM-EN-2.S, DM-RST-2.S, LOC-SQ-2.S, PROG-3.S, Q7.C, SOS-2.S, U1.GND
- net N$1: now also IC2A.Y; no longer U1.B1
- net N$10: now also IC2A.Y1, J1.TX; no longer Q1.E, RB-FTDI-2.1
- net N$11: now also IC2A.B; no longer Q1.B, Q2.B
- net N$12: now also IC2A.X2, LCD-1.S; no longer J1.TX, Q3.C
- net N$13: now also IC2A.A; no longer Q3.B, Q4.B
- net N$14: now also IC1.RB4/AN11/CPS4/COM0, U$1.5; no longer J1.RX, Q4.E
- net N$15: now also IC1.RB6/ICSPCLK/ICDCLK/SEG14, J2.PGC; no longer IC1.VPP/!MCLR!/RE3, PROG-1.S
- net N$16: now also J2.PGD; no longer PROG-4.S
- net N$17: now also R1.2, U$2.IN+; no longer IC1.RB6/ICSPCLK/ICDCLK/SEG14, PROG-5.S
- net N$2: now also IC2A.X; no longer Q5.C, U1.B2
- net N$21: now also DM-RST-1.1; no longer DM-RST-1.S
- net N$22: now also DM-EN-1.1; no longer DM-EN-1.S
- net N$23: now also SOS-1.1; no longer SOS-1.S
- net N$24: now also IC1.SEG12/VCAP/SS/SRNQ/C2OUT/C12IN0-/AN0/RA0, U$1.1; no longer LCD-1.S, Q5.E
- net N$26: now also IC1.RD6/CPS14/P1C/SEG19, R1.1; no longer Q6.G, Q7.E, R2.1
- net N$3: now also IC3.SCL
- net N$4: now also IC3.SDA
- net N$5: now also IC1.RD7/CPS15/P1D/SEG20, LOC-SQ-1.1; no longer IC1.RB4/AN11/CPS4/COM0, LOC-SQ-1.S
- net N$7: now also IC2A.X0, RB-FTDI-3.1; no longer Q2.E, Q3.E, U1.A1
- net N$8: now also IC2A.Y0, RB-FTDI-2.1; no longer Q1.C, Q4.C, U1.A2
- net N$9: now also IC2A.X1, J1.RX; no longer Q2.C, RB-FTDI-3.1
- net VPP: now also U$1.4, U$2.DC@2; no longer Q6.D
Other:
- moved on the sheet: DM-EN-1, DM-RST-1, LCD-1, LOC-SQ-1, R2, RB-FTDI-2, RB-FTDI-3, RB-INT-4, U$1
